File: msc_onlab106.brd (EAGLE design)
At the start: 127 x 85 mm, 134 parts, among them SW1 ENCODER_SW1-PEC12, SW2 ENCODER_SW1-PEC12, SW3 ENCODER_SW1-PEC12, U1 ATMEGA168, U2 ADUM1401BRWZ

Commit message: Values added
Parts:
- A1, A2, A3, A4, A5, F1, F2, F3, F4, N1, N10, N11, N12, N2, N3, N4, N5, N6, N7, N8, N9: value BUTTON_SMD -> TACTM-67N
- C2, C4: value (none) -> 22p
- D1, D2, D3, D4: value (none) -> TACTM-67N
- LCD: value TUXGR_16X2_R2 -> RC-1602-BB
- LCD_BACKLIGHT_FET: value (none) -> BSS 138
- LED17, LED18, LED19, LED20, LED21, LED22, LED23, LED24, LED25, LED26, LED27, LED28, LED29, LED30, LED31, LED32: value (none) -> OF-SMD 2012 R/Y/G
- R10, R11, R12, R13, R14, R17, R18, R19, R20, R21, R22, R23, R24, R7, R8, R9: value (none) -> 1k
- RESET: value BUTTON_SMD -> NSG 39-2
- TRIMPOT: value (none) -> 10k
- Y1: value (none) -> 16MHz
- renumbered DIS1 to LCD, JP1 to PROGRAMMING_CONNECTOR, L4941_5V to VOLTAGE_REGULATOR, Q1 to LCD_BACKLIGHT_FET, SW1 to E1, SW2 to E2, SW3 to E3, U$1 to A1, U$10 to A5, U$11 to N10, U$12 to N7, U$13 to F2, U$14 to F3, U$15 to F1, U$16 to A2, U$17 to N2, U$18 to N6, U$19 to N1, U$2 to N9, U$20 to N5, U$21 to F4, U$3 to N4, U$32 to TRIMPOT, U$39 to POWER_CONNECTOR, U$4 to A4, U$41 to RESET, U$42 to CONNECTOR, U$43 to DIP1, U$44 to DIP2, U$5 to N12, U$6 to N8, U$7 to A3, U$8 to N11, U$9 to N3, U1 to AVR, U2 to ADUM
